File: olimex-hx8k-pmod.sch (KiCad schematic (older format))
At the start: 11 parts, among them J1 Conn_02x20_Odd_Even_FPGA, J2 PMOD, J3 PMOD, J4 PMOD, J5 PMOD, SW1 SW_SPST, SW2 SW_SPST

Commit message: Move schematic symbols to project library
Signed-off-by: Rangel Ivanov <rangelivanov88@gmail.com>
Parts:
- C1, C2, C3, C4: symbol Device:C_Small -> my_lib:C_Small
- J1: symbol Connector_Generic:Conn_02x20_Odd_Even -> my_lib:Conn_02x20_Odd_Even
- J2, J3, J4, J5: symbol Connector_Generic:Conn_02x06_Top_Bottom -> my_lib:Conn_02x06_Top_Bottom
- SW1, SW2: symbol Switch:SW_SPST -> my_lib:SW_SPST
Changed lines of the file:
@@
 EESchema Schematic File Version 4
 LIBS:olimex-hx8k-pmod-cache
-EELAYER 29 0
+EELAYER 30 0
 EELAYER END
 $Descr A4 11693 8268
@@
 $EndDescr
 $Comp
-L Connector_Generic:Conn_02x20_Odd_Even J1
+L my_lib:Conn_02x20_Odd_Even J1
 U 1 1 5C93E121
 P 5525 3325
@@
 	4725 2525 4725 2325
 $Comp
-L power:+3.3V #PWR0102
+L my_lib:+3.3V #PWR0102
 U 1 1 5C8148DD
 P 4725 2325
@@
 	6125 2425 6175 2425
 $Comp
-L power:GND #PWR0103
+L my_lib:GND #PWR0103
 U 1 1 5C814A2B
 P 6175 2425
@@
 	4975 2925 5325 2925
 $Comp
-L Connector_Generic:Conn_02x06_Top_Bottom J2
+L my_lib:Conn_02x06_Top_Bottom J2
 U 1 1 5D48AA25
 P 3275 2475
@@
 $EndComp
 $Comp
-L power:+3.3V #PWR0104
+L my_lib:+3.3V #PWR0104
 U 1 1 5D48AA33
 P 3025 1875
@@
 $EndComp
 $Comp
-L power:+3.3V #PWR0105
+L my_lib:+3.3V #PWR0105
 U 1 1 5D48AA3D
 P 3625 1875
@@
 $EndComp
 $Comp
-L power:GND #PWR0106
+L my_lib:GND #PWR0106
 U 1 1 5D48AA4B
 P 2675 2875
@@
 $EndComp
 $Comp
-L power:GND #PWR0107
+L my_lib:GND #PWR0107
 U 1 1 5D48AA55
 P 3975 2875
@@
 	3625 2775 3575 2775
 $Comp
-L Device:C_Small C1
+L my_lib:C_Small C1
 U 1 1 5D5272A4
 P 2875 2775
@@
 	3025 2775 3075 2775
 $Comp
-L Connector_Generic:Conn_02x06_Top_Bottom J3
+L my_lib:Conn_02x06_Top_Bottom J3
 U 1 1 5D618DD9
 P 3275 4125
@@
 $EndComp
 $Comp
-L power:+3.3V #PWR0108
+L my_lib:+3.3V #PWR0108
 U 1 1 5D618DE3
 P 3025 3525
@@
 $EndComp
 $Comp
-L power:+3.3V #PWR0109
+L my_lib:+3.3V #PWR0109
 U 1 1 5D618DED
 P 3625 3525
@@
 $EndComp
 $Comp
-L power:GND #PWR0110
+L my_lib:GND #PWR0110
 U 1 1 5D618DF7
 P 2675 4525
@@
 	3625 4425 3575 4425
 $Comp
-L Device:C_Small C2
+L my_lib:C_Small C2
 U 1 1 5D618E21
 P 2875 4425
@@
 	5825 4225 6225 4225
 $Comp
-L Switch:SW_SPST SW1
+L my_lib:SW_SPST SW1
 U 1 1 5D6C7585
 P 4700 4325
@@
 	4900 4325 5325 4325
 $Comp
-L Switch:SW_SPST SW2
+L my_lib:SW_SPST SW2
 U 1 1 5D6D5B83
 P 6475 4325
@@
 	4500 4325 4500 4550
 $Comp
-L power:GND #PWR01
+L my_lib:GND #PWR01
 U 1 1 5D6E4F2A
 P 4500 4550
@@
 $EndComp
 $Comp
-L power:GND #PWR02
+L my_lib:GND #PWR02
 U 1 1 5D6E5DC3
 P 6675 4575
@@
 $EndComp
 $Comp
-L Connector_Generic:Conn_02x06_Top_Bottom J4
+L my_lib:Conn_02x06_Top_Bottom J4
 U 1 1 5D6E7EF8
 P 7525 2475
@@
 $EndComp
 $Comp
-L power:+3.3V #PWR05
+L my_lib:+3.3V #PWR05
 U 1 1 5D6E7F02
 P 7275 1875
@@
 $EndComp
 $Comp
-L power:+3.3V #PWR07
+L my_lib:+3.3V #PWR07
 U 1 1 5D6E7F0C
 P 7875 1875
@@
 $EndComp
 $Comp
-L power:GND #PWR03
+L my_lib:GND #PWR03
 U 1 1 5D6E7F16
 P 6925 2875
@@
 $EndComp
 $Comp
-L power:GND #PWR09
+L my_lib:GND #PWR09
 U 1 1 5D6E7F20
 P 8225 2875
@@
 	7875 2775 7825 2775
 $Comp
-L Device:C_Small C3
+L my_lib:C_Small C3
 U 1 1 5D6E7F3F
 P 7125 2775
@@
 PMOD2_8
 $Comp
-L Connector_Generic:Conn_02x06_Top_Bottom J5
+L my_lib:Conn_02x06_Top_Bottom J5
 U 1 1 5D6F2F93
 P 7575 4125
@@
 $EndComp
 $Comp
-L power:+3.3V #PWR06
+L my_lib:+3.3V #PWR06
 U 1 1 5D6F2F9D
 P 7325 3525
@@
 $EndComp
 $Comp
-L power:+3.3V #PWR08
+L my_lib:+3.3V #PWR08
 U 1 1 5D6F2FA7
 P 7925 3525
@@
 $EndComp
 $Comp
-L power:GND #PWR04
+L my_lib:GND #PWR04
 U 1 1 5D6F2FB1
 P 6975 4525
@@
 $EndComp
 $Comp
-L power:GND #PWR010
+L my_lib:GND #PWR010
 U 1 1 5D6F2FBB
 P 8275 4525
@@
 	7925 4425 7875 4425
 $Comp
-L Device:C_Small C4
+L my_lib:C_Small C4
 U 1 1 5D6F2FDA
 P 7175 4425
@@
 	4975 3925 5325 3925
 $Comp
-L power:PWR_FLAG #FLG0101
+L my_lib:PWR_FLAG #FLG0101
 U 1 1 5D721DCD
 P 2575 1775
@@
 	3025 1925 3025 2775
 $Comp
-L power:PWR_FLAG #FLG0102
+L my_lib:PWR_FLAG #FLG0102
 U 1 1 5D753869
 P 5175 2025
@@
 	5175 2425 4975 2425
 $Comp
-L power:PWR_FLAG #FLG0103
+L my_lib:PWR_FLAG #FLG0103
 U 1 1 5D762571
 P 2150 2750

Commit message: Rearrange pmod connections for easier routing
Add custom footprints for pmod connector and olimex expansion connector

Signed-off-by: Rangel Ivanov <rangelivanov88@gmail.com>
Parts:
- C1, C2, C3, C4: footprint (none) -> Capacitor_SMD:C_0805_2012Metric
- J1: footprint (none) -> olimex-hx8k-pmod:GPCB127SMT-02X20(YA-V36P-2X20-LF)
- J2, J3, J4, J5: footprint (none) -> olimex-hx8k-pmod:PinSocket_2x06_P2.54mm_Horizontal
- SW1, SW2: footprint (none) -> Button_Switch_THT:SW_PUSH_6mm
Changed lines of the file:
@@
 F 0 "J1" H 5575 4442 50  0000 C CNN
 F 1 "Conn_02x20_Odd_Even_FPGA" H 5575 4351 50  0000 C CNN
-F 2 "" H 5525 3325 50  0001 C CNN
+F 2 "olimex-hx8k-pmod:GPCB127SMT-02X20(YA-V36P-2X20-LF)" H 5525 3325 50  0001 C CNN
 F 3 "~" H 5525 3325 50  0001 C CNN
 	1    5525 3325
@@
 F 0 "J2" H 3325 2892 50  0000 C CNN
 F 1 "PMOD" H 3325 2801 50  0000 C CNN
-F 2 "" H 3275 2475 50  0001 C CNN
+F 2 "olimex-hx8k-pmod:PinSocket_2x06_P2.54mm_Horizontal" H 3275 2475 50  0001 C CNN
 F 3 "~" H 3275 2475 50  0001 C CNN
 	1    3275 2475
@@
 Wire Wire Line
 	3075 2575 2675 2575
-Text Label 2675 2275 0    50   ~ 0
+Text Label 2675 2575 0    50   ~ 0
 PMOD0_1
-Text Label 2675 2375 0    50   ~ 0
+Text Label 3975 2575 2    50   ~ 0
 PMOD0_2
 Text Label 2675 2475 0    50   ~ 0
 PMOD0_3
-Text Label 2675 2575 0    50   ~ 0
+Text Label 3975 2475 2    50   ~ 0
 PMOD0_4
 Text Label 4975 3525 0    50   ~ 0
@@
 Wire Wire Line
 	5325 4225 4975 4225
-Text Label 3975 2575 2    50   ~ 0
+Text Label 3975 2275 2    50   ~ 0
 PMOD0_8
-Text Label 3975 2475 2    50   ~ 0
+Text Label 2675 2275 0    50   ~ 0
 PMOD0_7
 Text Label 3975 2375 2    50   ~ 0
 PMOD0_6
-Text Label 3975 2275 2    50   ~ 0
+Text Label 2675 2375 0    50   ~ 0
 PMOD0_5
 Wire Wire Line
@@
 F 0 "C1" V 2975 2725 50  0000 L CNN
 F 1 "10n" V 3050 2700 50  0000 L CNN
-F 2 "" H 2875 2775 50  0001 C CNN
+F 2 "Capacitor_SMD:C_0805_2012Metric" H 2875 2775 50  0001 C CNN
 F 3 "~" H 2875 2775 50  0001 C CNN
 	1    2875 2775
@@
 F 0 "J3" H 3325 4542 50  0000 C CNN
 F 1 "PMOD" H 3325 4451 50  0000 C CNN
-F 2 "" H 3275 4125 50  0001 C CNN
+F 2 "olimex-hx8k-pmod:PinSocket_2x06_P2.54mm_Horizontal" H 3275 4125 50  0001 C CNN
 F 3 "~" H 3275 4125 50  0001 C CNN
 	1    3275 4125
@@
 Wire Wire Line
 	3075 4225 2675 4225
-Text Label 2675 3925 0    50   ~ 0
+Text Label 2675 4225 0    50   ~ 0
 PMOD1_1
-Text Label 2675 4025 0    50   ~ 0
+Text Label 3975 4225 2    50   ~ 0
 PMOD1_2
 Text Label 2675 4125 0    50   ~ 0
 PMOD1_3
-Text Label 2675 4225 0    50   ~ 0
+Text Label 3975 4125 2    50   ~ 0
 PMOD1_4
-Text Label 3975 4125 2    50   ~ 0
+Text Label 2675 3925 0    50   ~ 0
 PMOD1_7
 Text Label 3975 4025 2    50   ~ 0
 PMOD1_6
-Text Label 3975 3925 2    50   ~ 0
+Text Label 2675 4025 0    50   ~ 0
 PMOD1_5
 Wire Wire Line
@@
 F 0 "C2" V 2975 4375 50  0000 L CNN
 F 1 "10n" V 3050 4350 50  0000 L CNN
-F 2 "" H 2875 4425 50  0001 C CNN
+F 2 "Capacitor_SMD:C_0805_2012Metric" H 2875 4425 50  0001 C CNN
 F 3 "~" H 2875 4425 50  0001 C CNN
 	1    2875 4425
@@
 Wire Wire Line
 	2675 2675 2675 2875
-Text Label 3975 4225 2    50   ~ 0
+Text Label 3975 3925 2    50   ~ 0
 PMOD1_8
 Text Label 6225 2725 2    50   ~ 0
@@
 F 0 "SW1" H 4700 4560 50  0000 C CNN
 F 1 "SW_SPST" H 4700 4469 50  0000 C CNN
-F 2 "" H 4700 4325 50  0001 C CNN
+F 2 "Button_Switch_THT:SW_PUSH_6mm" H 4700 4325 50  0001 C CNN
 F 3 "~" H 4700 4325 50  0001 C CNN
 	1    4700 4325
@@
 F 0 "SW2" H 6475 4560 50  0000 C CNN
 F 1 "SW_SPST" H 6475 4469 50  0000 C CNN
-F 2 "" H 6475 4325 50  0001 C CNN
+F 2 "Button_Switch_THT:SW_PUSH_6mm" H 6475 4325 50  0001 C CNN
 F 3 "~" H 6475 4325 50  0001 C CNN
 	1    6475 4325
@@
 F 0 "J4" H 7575 2892 50  0000 C CNN
 F 1 "PMOD" H 7575 2801 50  0000 C CNN
-F 2 "" H 7525 2475 50  0001 C CNN
+F 2 "olimex-hx8k-pmod:PinSocket_2x06_P2.54mm_Horizontal" H 7525 2475 50  0001 C CNN
 F 3 "~" H 7525 2475 50  0001 C CNN
 	1    7525 2475
@@
 Text Label 6925 2275 0    50   ~ 0
 PMOD2_1
+Text Label 8225 2275 2    50   ~ 0
+PMOD2_2
 Text Label 6925 2375 0    50   ~ 0
-PMOD2_2
+PMOD2_3
+Text Label 8225 2375 2    50   ~ 0
+PMOD2_4
+Text Label 6925 2575 0    50   ~ 0
+PMOD2_7
+Text Label 8225 2475 2    50   ~ 0
+PMOD2_6
 Text Label 6925 2475 0    50   ~ 0
-PMOD2_3
-Text Label 6925 2575 0    50   ~ 0
-PMOD2_4
-Text Label 8225 2475 2    50   ~ 0
-PMOD2_7
-Text Label 8225 2375 2    50   ~ 0
-PMOD2_6
-Text Label 8225 2275 2    50   ~ 0
 PMOD2_5
 Wire Wire Line
@@
 F 0 "C3" V 7225 2725 50  0000 L CNN
 F 1 "10n" V 7300 2700 50  0000 L CNN
-F 2 "" H 7125 2775 50  0001 C CNN
+F 2 "Capacitor_SMD:C_0805_2012Metric" H 7125 2775 50  0001 C CNN
 F 3 "~" H 7125 2775 50  0001 C CNN
 	1    7125 2775
@@
 F 0 "J5" H 7625 4542 50  0000 C CNN
 F 1 "PMOD" H 7625 4451 50  0000 C CNN
-F 2 "" H 7575 4125 50  0001 C CNN
+F 2 "olimex-hx8k-pmod:PinSocket_2x06_P2.54mm_Horizontal" H 7575 4125 50  0001 C CNN
 F 3 "~" H 7575 4125 50  0001 C CNN
 	1    7575 4125
@@
 Text Label 6975 3925 0    50   ~ 0
 PMOD3_1
+Text Label 8275 3925 2    50   ~ 0
+PMOD3_2
 Text Label 6975 4025 0    50   ~ 0
-PMOD3_2
+PMOD3_3
+Text Label 8275 4025 2    50   ~ 0
+PMOD3_4
+Text Label 6975 4225 0    50   ~ 0
+PMOD3_7
+Text Label 8275 4125 2    50   ~ 0
+PMOD3_6
 Text Label 6975 4125 0    50   ~ 0
-PMOD3_3
-Text Label 6975 4225 0    50   ~ 0
-PMOD3_4
-Text Label 8275 4125 2    50   ~ 0
-PMOD3_7
-Text Label 8275 4025 2    50   ~ 0
-PMOD3_6
-Text Label 8275 3925 2    50   ~ 0
 PMOD3_5
 Wire Wire Line
@@
 F 0 "C4" V 7275 4375 50  0000 L CNN
 F 1 "10n" V 7350 4350 50  0000 L CNN
-F 2 "" H 7175 4425 50  0001 C CNN
+F 2 "Capacitor_SMD:C_0805_2012Metric" H 7175 4425 50  0001 C CNN
 F 3 "~" H 7175 4425 50  0001 C CNN
 	1    7175 4425
